File: Lyrebird Keyboard/Lyrebird Keyboard.kicad_pcb (KiCad board)
At the start: 4 copper layers, 95 parts, among them IC1 L7915CV, IC2 L78S15CV, IC3 MCP6022-E_SN, IC4 IR2113SPBF, IC5 IR2113SPBF, IC6 LM358DT, IC7 L7805ACD2T-TR, J1 WAV/ENV 4, J10 1776119-2, J11 1776119-2, J12 1776119-2, J13 MC-254-16-00-ST-DIP, J14 MC-254-16-00-ST-DIP, J15 MC-254-16-00-ST-DIP, J16 MC-254-16-00-ST-DIP, J17 MC-254-16-00-ST-DIP, J18 MC-254-16-00-ST-DIP, J19 MC-254-16-00-ST-DIP, J2 WAV/ENV 3, J20 1776119-2, J21 1776119-2, J3 WAV/ENV 2, J4 WAV/ENV 1, J5 TONE SRC 4, J6 TONE SRC 3, J7 TONE SRC 2, J8 TONE SRC 1, J9 1776119-2, Q1 BC848, Q2 BC848, Q3 IRFR2905ZTRPBF, Q4 IRFR2905ZTRPBF, Q5 IRFR2905ZTRPBF, Q6 IRFR2905ZTRPBF, U1 DF06S

Commit message: additional tracks laid
Parts:
- J11: value 1776119-2 -> 240V Out
- J12: value 1776119-2 -> 240V In
- J13, J14, J15, J16, J17, J18, J19: moved to B.Cu
- moved C23 244.3 mm to (235.1, 172.3), turned to 90 degrees
- moved C10 238.6 mm to (135.1, 182.3)
- moved C11 238.6 mm to (135.1, 185.7)
- moved C12 238.6 mm to (135.1, 189.0)
- moved C13 238.6 mm to (140.8, 179.0)
- moved C14 238.6 mm to (140.8, 182.3)
- moved C15 238.6 mm to (140.8, 185.7)
- moved C17 238.6 mm to (140.8, 189.0)
- moved C19 238.6 mm to (146.4, 179.0)
- moved C20 238.6 mm to (146.4, 182.3)
- moved C26 238.6 mm to (146.4, 185.7)
- moved C28 238.6 mm to (146.4, 189.0)
- moved C6 238.6 mm to (123.0, 181.1)
- moved C7 238.6 mm to (123.0, 186.5)
- moved C8 238.6 mm to (123.0, 192.0)
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Routing:
- net C#33: track 0.00 -> 91.2 mm
- net D34: track 0.00 -> 91.1 mm
- net C#9: track 0.00 -> 81.9 mm
- net G3: track 0.00 -> 81.8 mm
- net F25: track 0.00 -> 81.8 mm
- net B7: track 0.00 -> 81.7 mm
- net B19: track 0.00 -> 81.7 mm
- net F1: track 0.00 -> 81.7 mm
- net B31: track 0.00 -> 81.7 mm
- net G27: track 0.00 -> 81.6 mm
- net E60: track 0.00 -> 81.6 mm
- net A29: track 0.00 -> 81.6 mm
- net C#21: track 0.00 -> 81.6 mm
- net D#23: track 0.00 -> 81.6 mm
- net D#11: track 0.00 -> 81.6 mm
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