File: Lyrebird Keyboard/Lyrebird Keyboard.kicad_pcb (KiCad board)
At the start: 4 copper layers, 95 parts, among them IC1 L7915CV, IC2 L78S15CV, IC3 MCP6022-E_SN, IC4 IR2113SPBF, IC5 IR2113SPBF, IC6 LM358DT, IC7 L7805ACD2T-TR, J1 WAV/ENV 4, J10 AC IN 2, J11 240V Out, J12 240 In, J13 MC-254-16-00-ST-DIP, J14 MC-254-16-00-ST-DIP, J15 MC-254-16-00-ST-DIP, J16 MC-254-16-00-ST-DIP, J17 MC-254-16-00-ST-DIP, J18 MC-254-16-00-ST-DIP, J19 MC-254-16-00-ST-DIP, J2 WAV/ENV 3, J20 AMP Out, J21 SUB Out, J3 WAV/ENV 2, J4 WAV/ENV 1, J5 TONE SRC 4, J6 TONE SRC 3, J7 TONE SRC 2, J8 TONE SRC 1, J9 AC IN 1, Q1 BC848, Q2 BC848, Q3 IRFR2905ZTRPBF, Q4 IRFR2905ZTRPBF, Q5 IRFR2905ZTRPBF, Q6 IRFR2905ZTRPBF, U1 DF06S

Commit message: Tracks almost finished
Parts:
- added J22: Square Test, Connector_PinHeader_2.54mm:PinHeader_1x01_P2.54mm_Vertical, F.Cu at (175.7, 141.6)
- added J23: Bias Test Point 2, Connector_PinHeader_2.54mm:PinHeader_1x01_P2.54mm_Vertical, F.Cu at (227.8, 139.3)
- added J24: Bias Test Point 1, Connector_PinHeader_2.54mm:PinHeader_1x01_P2.54mm_Vertical, F.Cu at (216.0, 139.3)
- J19: value MC-254-16-00-ST-DIP -> Triangle Test; footprint SamacSys_Parts:SHDR16W64P254_2X8_2798X910X910P -> Connector_PinHeader_2.54mm:PinHeader_1x01_P2.54mm_Vertical; moved to F.Cu
- moved J20 172.8 mm to (85.8, 165.7)
- moved J21 146.8 mm to (98.8, 165.8)
- moved IC4 136.4 mm to (213.3, 157.2)
- moved C19 124.5 mm to (149.1, 141.0), turned to -90 degrees
- moved C26 124.5 mm to (149.0, 148.1), turned to 90 degrees
- moved L1 121.5 mm to (141.1, 139.0), turned to -90 degrees
- moved L2 114.8 mm to (141.1, 150.1), turned to 90 degrees
- moved Q3 114.3 mm to (192.5, 167.1), turned to 90 degrees
- moved Q4 111.9 mm to (207.9, 167.0), turned to -90 degrees
- moved R13 110.2 mm to (180.2, 142.3)
- moved R16 107.3 mm to (183.9, 149.1), turned to 90 degrees
- moved J19 100.6 mm to (200.4, 146.8), turned to 0 degrees
- moved IC5 99.5 mm to (213.3, 131.7)
- moved R12 97.2 mm to (189.4, 150.2), turned to 180 degrees
- moved C23 93.3 mm to (142.2, 164.1), turned to -90 degrees
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Connections:
- J1 pad A5: +30V -> GND
- J1 pad A6: +30V -> GND
- J13 pad 1: F1 -> GND
- J13 pad 10: E12 -> C8
- J13 pad 11: A#6 -> C#9
- J13 pad 12: D#11 -> D10
- J13 pad 13: B7 -> D#11
- J13 pad 14: D10 -> E12
- J13 pad 15: C8 -> F13
- J13 pad 16: C#9 -> F#14
- J13 pad 3: F#2 -> F1
- J13 pad 4: +30V -> F#2
- J13 pad 6: GND -> G#4
- J13 pad 7: G#4 -> A5
- J13 pad 8: GND -> A#6
- J13 pad 9: A5 -> B7
- J14 pad 1: F13 -> GND
- J14 pad 10: E24 -> D22
- J14 pad 11: A#18 -> D#23
- J14 pad 12: D#23 -> E24
- J14 pad 13: B19 -> F25
- J14 pad 14: D22 -> F#26
- J14 pad 15: C20 -> G27
- J14 pad 16: C#21 -> G#28
- J14 pad 3: F#14 -> G15
- J14 pad 4: +30V -> G#16
- J14 pad 5: G15 -> A17
- J14 pad 6: GND -> A#18
- J14 pad 7: G#16 -> B19
- J14 pad 8: GND -> C20
- J14 pad 9: A17 -> C#21
- J15 pad 1: F25 -> GND
- J15 pad 10: E36 -> unconnected-(J15-Pad10)
- J15 pad 11: A#30 -> unconnected-(J15-Pad11)
- J15 pad 12: D#35 -> unconnected-(J15-Pad12)
- J15 pad 13: B31 -> unconnected-(J15-Pad13)
- J15 pad 14: D34 -> unconnected-(J15-Pad14)
- J15 pad 15: C32 -> unconnected-(J15-Pad15)
- J15 pad 16: C#33 -> unconnected-(J15-Pad16)
- J15 pad 3: F#26 -> A29
- J15 pad 4: +30V -> A#30
- J15 pad 5: G27 -> B31
- J15 pad 6: GND -> C32
- J15 pad 7: G#28 -> C#33
- J15 pad 8: GND -> unconnected-(J15-Pad8)
- J15 pad 9: A29 -> unconnected-(J15-Pad9)
- J16 pad 1: F37 -> GND
- J16 pad 10: E48 -> F#38
- J16 pad 11: A#42 -> A41
- J16 pad 12: D#47 -> G#40
- J16 pad 14: D46 -> A#42
- J16 pad 15: C44 -> C#45
- J16 pad 16: C#45 -> C44
- J16 pad 3: F#38 -> unconnected-(J16-Pad3)
- J16 pad 4: +30V -> unconnected-(J16-Pad4)
- J16 pad 5: G39 -> D#35
- J16 pad 6: GND -> D34
- J16 pad 7: G#40 -> F37
- J16 pad 8: GND -> E36
- J16 pad 9: A41 -> G39
- J17 pad 1: F49 -> GND
- J17 pad 10: E60 -> G#52
- J17 pad 11: A#54 -> B55
- J17 pad 12: D#59 -> A#54
- J17 pad 13: B55 -> C#57
- J17 pad 14: D58 -> C56
- J17 pad 15: C56 -> D#59
- J17 pad 16: C#57 -> D58
- J17 pad 3: F#50 -> D#47
- J17 pad 4: +30V -> D46
- J17 pad 5: G51 -> F49
- J17 pad 6: GND -> E48
- J17 pad 7: G#52 -> G51
- J17 pad 8: GND -> F#50
- J18 pad 1: F61 -> GND
- J18 pad 10: E72 -> A#66
- J18 pad 11: A#66 -> C#69
- J18 pad 12: D#71 -> C68
- J18 pad 13: B67 -> D#71
- J18 pad 15: C68 -> F73
- J18 pad 16: C#69 -> E72
- J18 pad 3: F#62 -> F61
- J18 pad 4: +30V -> E60
- J18 pad 6: GND -> F#62
- J18 pad 7: G#64 -> A65
- J18 pad 8: GND -> G#64
- J18 pad 9: A65 -> B67
- J19 pad 1: F73 -> TRI WAVE OUT
- J2 pad A5: +30V -> GND
- J2 pad A6: +30V -> GND
- J3 pad A5: +30V -> GND
- J3 pad A6: +30V -> GND
- J4 pad A5: +30V -> GND
- J4 pad A6: +30V -> GND
- J5 pad A5: +30V -> GND
- J5 pad A6: +30V -> GND
- J6 pad A5: +30V -> GND
- J6 pad A6: +30V -> GND
- J7 pad A5: +30V -> GND
- J7 pad A6: +30V -> GND
- J8 pad A5: +30V -> GND
- J8 pad A6: +30V -> GND
Routing:
- net +30V: track 55.4 -> 381.0 mm
- net +5V: track 0.00 -> 241.2 mm, vias 0 -> 4
- net +15V: track 29.7 -> 266.2 mm, vias 0 -> 2
- net GND: track 238.7 -> 430.5 mm
- net VS2: track 0.00 -> 101.2 mm
- net +VED: track 183.4 -> 278.2 mm
- net VS1: track 0.00 -> 94.4 mm
- net LINE OUT: track 183.4 -> 271.9 mm
- net AMP OUT: track 0.00 -> 86.2 mm
- net D#35: track 78.5 -> 155.9 mm
- net F37: track 78.6 -> 155.4 mm
- net G39: track 78.6 -> 155.0 mm
- net B43: track 78.6 -> 154.5 mm
- net A41: track 78.5 -> 154.0 mm
- net C#45: track 78.5 -> 153.0 mm
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- added copper zone on In1.Cu, net +15V
- added copper zone on B.Cu, net +30V
- added copper zone on In2.Cu, net -15V
- added copper zone on F.Cu, net GND
Other:
- board outline added: 220.1 x 160.3 mm
- board text added: "OSC Adj."

Commit message: Mainboard Complete
Parts:
- added J25: Pedals, SamacSys_Parts:CTB05083, F.Cu at (24.3, 137.1)
- J1: value WAV/ENV 4 -> WAV/ENV 4 (MIDI)
- J13: value MC-254-16-00-ST-DIP -> Keys 1 to 14
- J14: value MC-254-16-00-ST-DIP -> Keys 15 to 28
- J15: value MC-254-16-00-ST-DIP -> Keys 29 to 33
- J16: value MC-254-16-00-ST-DIP -> Keys 34 to 45
- J17: value MC-254-16-00-ST-DIP -> Keys 46 to 59
- J18: value MC-254-16-00-ST-DIP -> Keys 60 to 73
- moved Q2 12.1 mm to (209.6, 152.3)
- moved R3 12.1 mm to (209.9, 148.1)
- moved C9 11.8 mm to (214.1, 151.5)
- moved J23 11.8 mm to (216.2, 137.4)
- moved R15 11.8 mm to (186.2, 158.3)
- moved VR3 11.8 mm to (214.5, 120.7)
- moved Z2 11.8 mm to (163.6, 145.5)
- moved C7 11.8 mm to (67.4, 89.7)
- moved J21 11.8 mm to (87.2, 163.8)
- moved C4 11.8 mm to (40.3, 147.3)
- moved J9 11.8 mm to (48.2, 163.8)
- moved U1 11.8 mm to (57.2, 151.7)
- moved J7 11.8 mm to (58.1, 22.9)
- moved C1 11.8 mm to (67.8, 147.3)
- moved C13 11.8 mm to (181.6, 156.5)
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Connections:
- J1 pad A6: GND -> +30V
Routing:
- net SUSTAIN: track 183.4 -> 305.7 mm
- net +VT: track 222.0 -> 336.9 mm
- net SOFT: track 183.4 -> 297.4 mm
- net GND: track 430.5 -> 439.8 mm, vias 0 -> 4
- net +5V: track 241.2 -> 242.6 mm
- net +VED: track 278.2 -> 279.4 mm
- net Net-(IC6-IN2-): track 24.6 -> 25.5 mm
- net B43: track 154.5 -> 153.7 mm
Other:
- outline, holes or cut-outs redrawn
