File: Lyrebird Keyboard/_autosave-Lyrebird Keyboard.kicad_sch (KiCad schematic)
At the start: 99 parts, among them IC1 L7915CV, IC2 L78S15CV, IC3 MCP6022-E_SN, IC4 IR2113SPBF, IC5 IR2113SPBF, IC6 LM358DT, IC7 L7805ACD2T-TR, J1 WAV/ENV 4 (MIDI), J10 AC IN 2, J11 240V Out, J12 240 In, J13 Keys 1 to 14, J14 Keys 15 to 28, J15 Keys 29 to 33, J16 Keys 34 to 45, J17 Keys 46 to 59, J18 Keys 60 to 73, J19 Triangle Test, J2 WAV/ENV 3, J20 AMP Out, J21 SUB Out, J22 Square Test, J23 Bias Test Point 2, J24 Bias Test Point 1, J25 Pedals, J3 WAV/ENV 2, J4 WAV/ENV 1, J5 TONE SRC 4, J6 TONE SRC 3, J7 TONE SRC 2, J8 TONE SRC 1, J9 AC IN 1, Q1 BC848, Q2 BC848, Q3 IRFR2905ZTRPBF, Q4 IRFR2905ZTRPBF, Q5 IRFR2905ZTRPBF, Q6 IRFR2905ZTRPBF, U1 DF06S

Commit message: Major Design Changes
Completed Tone Generator Board, board now only provides base notes, individual notes will be generated on the wave shaping boards.

Made major changes to pci slot config, and have increased grounding of the slots.

May need decoupling capacitors on tone generator board, but tight for room
Connections:
- net +15V: now also J2.A17, J2.A3, J2.B17, J2.B3, J3.A17, J3.A3, J3.B17, J3.B3, J4.A17, J4.A3, J4.B17, J4.B3, J5.A17, J5.A3, J5.B17, J5.B3, J6.A17, J6.A3, J6.B17, J6.B3, J7.A17, J7.A3, J7.B17, J7.B3, J8.A17, J8.A3, J8.B17, J8.B3; no longer J1.A18, J1.A4, J2.A18, J2.A4, J2.B18, J2.B4, J3.A18, J3.A4, J3.B18, J3.B4, J4.A18, J4.A4, J4.B18, J4.B4, J5.A18, J5.A4, J5.B18, J5.B4, J6.A18, J6.A4, J6.B18, J6.B4, J7.A18, J7.A4, J7.B18, J7.B4, J8.A18, J8.A4, J8.B18, J8.B4
- net +30V: now also J2.A1, J2.A15, J2.B1, J2.B15, J3.A1, J3.A15, J3.B1, J3.B15, J4.A1, J4.A15, J4.B1, J4.B15, J5.A1, J5.A15, J5.B1, J5.B15, J6.A1, J6.A15, J6.B1, J6.B15, J7.A1, J7.A15, J7.B1, J7.B15, J8.A1, J8.A15, J8.B1, J8.B15; no longer J1.A16, J1.A2, J2.A16, J2.A2, J2.B16, J2.B2, J3.A16, J3.A2, J3.B16, J3.B2, J4.A16, J4.A2, J4.B16, J4.B2, J5.A16, J5.A2, J5.B16, J5.B2, J6.A16, J6.A2, J6.B16, J6.B2, J7.A16, J7.A2, J7.B16, J7.B2, J8.A16, J8.A2, J8.B16, J8.B2
- net +VED: now also J2.B7, J3.B7, J4.B7, J5.B7, J6.B7, J7.B7, J8.B7; no longer J2.B8, J3.B8, J4.B8, J5.B8, J6.B8, J7.B8, J8.B8
- net +VT: now also J2.A7, J3.A7, J4.A7, J5.A7, J6.A7, J7.A7, J8.A7; no longer J1.A8, J2.A8, J3.A8, J4.A8, J5.A8, J6.A8, J7.A8, J8.A8
- net -15V: now also J2.A19, J2.A5, J2.B19, J2.B5, J3.A19, J3.A5, J3.B19, J3.B5, J4.A19, J4.A5, J4.B19, J4.B5, J5.A19, J5.A5, J5.B19, J5.B5, J6.A19, J6.A5, J6.B19, J6.B5, J7.A19, J7.A5, J7.B19, J7.B5, J8.A19, J8.A5, J8.B19, J8.B5; no longer J1.A20, J1.A6, J2.A20, J2.A6, J2.B20, J2.B6, J3.A20, J3.A6, J3.B20, J3.B6, J4.A20, J4.A6, J4.B20, J4.B6, J5.A20, J5.A6, J5.B20, J5.B6, J6.A20, J6.A6, J6.B20, J6.B6, J7.A20, J7.A6, J7.B20, J7.B6, J8.A20, J8.A6, J8.B20, J8.B6
- net EXP 1: now also J2.A33, J3.A33, J4.A33, J5.A33, J6.A33, J7.A33, J8.A33; no longer J1.A34, J2.A34, J3.A34, J4.A34, J5.A34, J6.A34, J7.A34, J8.A34
- net EXP 11: now also J2.B39, J3.B39, J4.B39, J5.B39, J6.B39, J7.B39, J8.B39; no longer J2.B40, J3.B40, J4.B40, J5.B40, J6.B40, J7.B40, J8.B40
- net EXP 12: now also J2.B41, J3.B41, J4.B41, J5.B41, J6.B41, J7.B41, J8.B41; no longer J2.B42, J3.B42, J4.B42, J5.B42, J6.B42, J7.B42, J8.B42
- net EXP 13: now also J2.B43, J3.B43, J4.B43, J5.B43, J6.B43, J7.B43, J8.B43; no longer J2.B44, J3.B44, J4.B44, J5.B44, J6.B44, J7.B44, J8.B44
- net EXP 2: now also J2.A35, J3.A35, J4.A35, J5.A35, J6.A35, J7.A35, J8.A35; no longer J1.A36, J2.A36, J3.A36, J4.A36, J5.A36, J6.A36, J7.A36, J8.A36
- net EXP 3: now also J2.A37, J3.A37, J4.A37, J5.A37, J6.A37, J7.A37, J8.A37; no longer J1.A38, J2.A38, J3.A38, J4.A38, J5.A38, J6.A38, J7.A38, J8.A38
- net EXP 4: now also J2.A39, J3.A39, J4.A39, J5.A39, J6.A39, J7.A39, J8.A39; no longer J1.A40, J2.A40, J3.A40, J4.A40, J5.A40, J6.A40, J7.A40, J8.A40
- net EXP 5: now also J2.A41, J3.A41, J4.A41, J5.A41, J6.A41, J7.A41, J8.A41; no longer J1.A42, J2.A42, J3.A42, J4.A42, J5.A42, J6.A42, J7.A42, J8.A42
- net EXP 6: now also J2.A43, J3.A43, J4.A43, J5.A43, J6.A43, J7.A43, J8.A43; no longer J1.A44, J2.A44, J3.A44, J4.A44, J5.A44, J6.A44, J7.A44, J8.A44
- net EXP 7: now also J2.A45, J3.A45, J4.A45, J5.A45, J6.A45, J7.A45, J8.A45; no longer J1.A46, J2.A46, J3.A46, J4.A46, J5.A46, J6.A46, J7.A46, J8.A46
- net EXP10: now also J2.B37, J3.B37, J4.B37, J5.B37, J6.B37, J7.B37, J8.B37; no longer J2.B38, J3.B38, J4.B38, J5.B38, J6.B38, J7.B38, J8.B38
- net EXP8: now also J2.B33, J3.B33, J4.B33, J5.B33, J6.B33, J7.B33, J8.B33; no longer J2.B34, J3.B34, J4.B34, J5.B34, J6.B34, J7.B34, J8.B34
- net EXP9: now also J2.B35, J3.B35, J4.B35, J5.B35, J6.B35, J7.B35, J8.B35; no longer J2.B36, J3.B36, J4.B36, J5.B36, J6.B36, J7.B36, J8.B36
- net GND: now also J1.A10, J1.A12, J1.A14, J1.A16, J1.A18, J1.A2, J1.A20, J1.A22, J1.A24, J1.A26, J1.A28, J1.A30, J1.A32, J1.A34, J1.A36, J1.A38, J1.A4, J1.A40, J1.A42, J1.A44, J1.A46, J1.A6, J1.A8, J2.A10, J2.A12, J2.A14, J2.A16, J2.A18, J2.A2, J2.A20, J2.A22, J2.A24, J2.A26, J2.A28, J2.A30, J2.A32, J2.A34, J2.A36, J2.A38, J2.A4, J2.A40, J2.A42, J2.A44, J2.A46, J2.A6, J2.A8, J2.B10, J2.B12, J2.B14, J2.B16, J2.B18, J2.B2, J2.B20, J2.B22, J2.B24, J2.B26, J2.B28, J2.B30, J2.B32, J2.B34, J2.B36, J2.B38, J2.B4, J2.B40, J2.B42, J2.B44, J2.B6, J2.B8, J3.A10, J3.A12, J3.A14, J3.A16, J3.A18, J3.A2, J3.A20, J3.A22, J3.A24, J3.A26, J3.A28, J3.A30, J3.A32, J3.A34, J3.A36, J3.A38, J3.A4, J3.A40, J3.A42, J3.A44, J3.A46, J3.A6, J3.A8, J3.B10, J3.B12, J3.B14, J3.B16, J3.B18, J3.B2, J3.B20, J3.B22, J3.B24, J3.B26, J3.B28, J3.B30, J3.B32, J3.B34, J3.B36, J3.B38, J3.B4, J3.B40, J3.B42, J3.B44, J3.B6, J3.B8, J4.A10, J4.A12, J4.A14, J4.A16, J4.A18, J4.A2, J4.A20, J4.A22, J4.A24, J4.A26, J4.A28, J4.A30, J4.A32, J4.A34, J4.A36, J4.A38, J4.A4, J4.A40, J4.A42, J4.A44, J4.A46, J4.A6, J4.A8, J4.B10, J4.B12, J4.B14, J4.B16, J4.B18, J4.B2, J4.B20, J4.B22, J4.B24, J4.B26, J4.B28, J4.B30, J4.B32, J4.B34, J4.B36, J4.B38, J4.B4, J4.B40, J4.B42, J4.B44, J4.B6, J4.B8, J5.A10, J5.A12, J5.A14, J5.A16, J5.A18, J5.A2, J5.A20, J5.A22, J5.A24, J5.A26, J5.A28, J5.A30, J5.A32, J5.A34, J5.A36, J5.A38, J5.A4, J5.A40, J5.A42, J5.A44, J5.A46, J5.A48, J5.A6, J5.A8, J5.B10, J5.B12, J5.B14, J5.B16, J5.B18, J5.B2, J5.B20, J5.B22, J5.B24, J5.B26, J5.B28, J5.B30, J5.B32, J5.B34, J5.B36, J5.B38, J5.B4, J5.B40, J5.B42, J5.B44, J5.B46, J5.B48, J5.B6, J5.B8, J6.A10, J6.A12, J6.A14, J6.A16, J6.A18, J6.A2, J6.A20, J6.A22, J6.A24, J6.A26, J6.A28, J6.A30, J6.A32, J6.A34, J6.A36, J6.A38, J6.A4, J6.A40, J6.A42, J6.A44, J6.A46, J6.A48, J6.A6, J6.A8, J6.B10, J6.B12, J6.B14, J6.B16, J6.B18, J6.B2, J6.B20, J6.B22, J6.B24, J6.B26, J6.B28, J6.B30, J6.B32, J6.B34, J6.B36, J6.B38, J6.B4, J6.B40, J6.B42, J6.B44, J6.B46, J6.B48, J6.B6, J6.B8, J7.A10, J7.A12, J7.A14, J7.A16, J7.A18, J7.A2, J7.A20, J7.A22, J7.A24, J7.A26, J7.A28, J7.A30, J7.A32, J7.A34, J7.A36, J7.A38, J7.A4, J7.A40, J7.A42, J7.A44, J7.A46, J7.A48, J7.A6, J7.A8, J7.B10, J7.B12, J7.B14, J7.B16, J7.B18, J7.B2, J7.B20, J7.B22, J7.B24, J7.B26, J7.B28, J7.B30, J7.B32, J7.B34, J7.B36, J7.B38, J7.B4, J7.B40, J7.B42, J7.B44, J7.B46, J7.B48, J7.B6, J7.B8, J8.A10, J8.A12, J8.A14, J8.A16, J8.A18, J8.A2, J8.A20, J8.A22, J8.A24, J8.A26, J8.A28, J8.A30, J8.A32, J8.A34, J8.A36, J8.A38, J8.A4, J8.A40, J8.A42, J8.A44, J8.A46, J8.A48, J8.A6, J8.A8, J8.B10, J8.B12, J8.B14, J8.B16, J8.B18, J8.B2, J8.B20, J8.B22, J8.B24, J8.B26, J8.B28, J8.B30, J8.B32, J8.B34, J8.B36, J8.B38, J8.B4, J8.B40, J8.B42, J8.B44, J8.B46, J8.B48, J8.B6, J8.B8; no longer J1.A1, J1.A11, J1.A13, J1.A15, J1.A17, J1.A19, J1.A21, J1.A23, J1.A25, J1.A27, J1.A29, J1.A3, J1.A31, J1.A33, J1.A35, J1.A37, J1.A39, J1.A41, J1.A43, J1.A45, J1.A5, J1.A7, J1.A9, J2.A1, J2.A11, J2.A13, J2.A15, J2.A17, J2.A19, J2.A21, J2.A23, J2.A25, J2.A27, J2.A29, J2.A3, J2.A31, J2.A33, J2.A35, J2.A37, J2.A39, J2.A41, J2.A43, J2.A45, J2.A5, J2.A7, J2.A9, J2.B1, J2.B11, J2.B13, J2.B15, J2.B17, J2.B19, J2.B21, J2.B23, J2.B25, J2.B27, J2.B29, J2.B3, J2.B31, J2.B33, J2.B35, J2.B37, J2.B39, J2.B41, J2.B43, J2.B45, J2.B5, J2.B7, J2.B9, J3.A1, J3.A11, J3.A13, J3.A15, J3.A17, J3.A19, J3.A21, J3.A23, J3.A25, J3.A27, J3.A29, J3.A3, J3.A31, J3.A33, J3.A35, J3.A37, J3.A39, J3.A41, J3.A43, J3.A45, J3.A5, J3.A7, J3.A9, J3.B1, J3.B11, J3.B13, J3.B15, J3.B17, J3.B19, J3.B21, J3.B23, J3.B25, J3.B27, J3.B29, J3.B3, J3.B31, J3.B33, J3.B35, J3.B37, J3.B39, J3.B41, J3.B43, J3.B45, J3.B5, J3.B7, J3.B9, J4.A1, J4.A11, J4.A13, J4.A15, J4.A17, J4.A19, J4.A21, J4.A23, J4.A25, J4.A27, J4.A29, J4.A3, J4.A31, J4.A33, J4.A35, J4.A37, J4.A39, J4.A41, J4.A43, J4.A45, J4.A5, J4.A7, J4.A9, J4.B1, J4.B11, J4.B13, J4.B15, J4.B17, J4.B19, J4.B21, J4.B23, J4.B25, J4.B27, J4.B29, J4.B3, J4.B31, J4.B33, J4.B35, J4.B37, J4.B39, J4.B41, J4.B43, J4.B45, J4.B5, J4.B7, J4.B9, J5.A1, J5.A11, J5.A13, J5.A15, J5.A17, J5.A19, J5.A21, J5.A23, J5.A25, J5.A27, J5.A29, J5.A3, J5.A31, J5.A33, J5.A35, J5.A37, J5.A39, J5.A41, J5.A43, J5.A45, J5.A47, J5.A49, J5.A5, J5.A7, J5.A9, J5.B1, J5.B11, J5.B13, J5.B15, J5.B17, J5.B19, J5.B21, J5.B23, J5.B25, J5.B27, J5.B29, J5.B3, J5.B31, J5.B33, J5.B35, J5.B37, J5.B39, J5.B41, J5.B43, J5.B45, J5.B47, J5.B49, J5.B5, J5.B7, J5.B9, J6.A1, J6.A11, J6.A13, J6.A15, J6.A17, J6.A19, J6.A21, J6.A23, J6.A25, J6.A27, J6.A29, J6.A3, J6.A31, J6.A33, J6.A35, J6.A37, J6.A39, J6.A41, J6.A43, J6.A45, J6.A47, J6.A49, J6.A5, J6.A7, J6.A9, J6.B1, J6.B11, J6.B13, J6.B15, J6.B17, J6.B19, J6.B21, J6.B23, J6.B25, J6.B27, J6.B29, J6.B3, J6.B31, J6.B33, J6.B35, J6.B37, J6.B39, J6.B41, J6.B43, J6.B45, J6.B47, J6.B49, J6.B5, J6.B7, J6.B9, J7.A1, J7.A11, J7.A13, J7.A15, J7.A17, J7.A19, J7.A21, J7.A23, J7.A25, J7.A27, J7.A29, J7.A3, J7.A31, J7.A33, J7.A35, J7.A37, J7.A39, J7.A41, J7.A43, J7.A45, J7.A47, J7.A49, J7.A5, J7.A7, J7.A9, J7.B1, J7.B11, J7.B13, J7.B15, J7.B17, J7.B19, J7.B21, J7.B23, J7.B25, J7.B27, J7.B29, J7.B3, J7.B31, J7.B33, J7.B35, J7.B37, J7.B39, J7.B41, J7.B43, J7.B45, J7.B47, J7.B49, J7.B5, J7.B7, J7.B9, J8.A1, J8.A11, J8.A13, J8.A15, J8.A17, J8.A19, J8.A21, J8.A23, J8.A25, J8.A27, J8.A29, J8.A3, J8.A31, J8.A33, J8.A35, J8.A37, J8.A39, J8.A41, J8.A43, J8.A45, J8.A47, J8.A49, J8.A5, J8.A7, J8.A9, J8.B1, J8.B11, J8.B13, J8.B15, J8.B17, J8.B19, J8.B21, J8.B23, J8.B25, J8.B27, J8.B29, J8.B3, J8.B31, J8.B33, J8.B35, J8.B37, J8.B39, J8.B41, J8.B43, J8.B45, J8.B47, J8.B49, J8.B5, J8.B7, J8.B9
- net LINE OUT: now also J2.B13, J3.B13, J4.B13, J5.B13, J6.B13, J7.B13, J8.B13; no longer J2.B14, J3.B14, J4.B14, J5.B14, J6.B14, J7.B14, J8.B14
- net SELECT 1: now also J2.B45, J3.B45, J4.B45, J5.B45, J6.B45, J7.B45, J8.B45; no longer J5.B46, J6.B46, J7.B46, J8.B46
- net SELECT 2: now also J5.B47, J6.B47, J7.B47, J8.B47; no longer J5.B48, J6.B48, J7.B48, J8.B48
- net SELECT 3: now also J5.B49, J6.B49, J7.B49, J8.B49; no longer J5.A48, J6.A48, J7.A48, J8.A48
- net SELECT 4: now also J5.A47, J6.A47, J7.A47, J8.A47; no longer J1.A10, J2.A10, J3.A10, J4.A10, J5.A10, J6.A10, J7.A10, J8.A10
- net SELECT 5: now also J5.A49, J6.A49, J7.A49, J8.A49; no longer J1.A12, J2.A12, J3.A12, J4.A12, J5.A12, J6.A12, J7.A12, J8.A12
- net SELECT 6: now also J2.A9, J3.A9, J4.A9, J5.A9, J6.A9, J7.A9, J8.A9; no longer J1.A14, J2.A14, J3.A14, J4.A14, J5.A14, J6.A14, J7.A14, J8.A14
- net SOFT: now also J2.B11, J3.B11, J4.B11, J5.B11, J6.B11, J7.B11, J8.B11; no longer J2.B12, J3.B12, J4.B12, J5.B12, J6.B12, J7.B12, J8.B12
- net SUSTAIN: now also J2.B9, J3.B9, J4.B9, J5.B9, J6.B9, J7.B9, J8.B9; no longer J2.B10, J3.B10, J4.B10, J5.B10, J6.B10, J7.B10, J8.B10
- net TONE 1: now also J2.A21, J3.A21, J4.A21, J5.A21, J6.A21, J7.A21, J8.A21; no longer J1.A22, J2.A22, J3.A22, J4.A22, J5.A22, J6.A22, J7.A22, J8.A22
- net TONE 10: now also J2.B27, J3.B27, J4.B27, J5.B27, J6.B27, J7.B27, J8.B27; no longer J2.B28, J3.B28, J4.B28, J5.B28, J6.B28, J7.B28, J8.B28
- net TONE 11: now also J2.B29, J3.B29, J4.B29, J5.B29, J6.B29, J7.B29, J8.B29; no longer J2.B30, J3.B30, J4.B30, J5.B30, J6.B30, J7.B30, J8.B30
- net TONE 12: now also J2.B31, J3.B31, J4.B31, J5.B31, J6.B31, J7.B31, J8.B31; no longer J2.B32, J3.B32, J4.B32, J5.B32, J6.B32, J7.B32, J8.B32
- net TONE 2: now also J2.A23, J3.A23, J4.A23, J5.A23, J6.A23, J7.A23, J8.A23; no longer J1.A24, J2.A24, J3.A24, J4.A24, J5.A24, J6.A24, J7.A24, J8.A24
- net TONE 3: now also J2.A25, J3.A25, J4.A25, J5.A25, J6.A25, J7.A25, J8.A25; no longer J1.A26, J2.A26, J3.A26, J4.A26, J5.A26, J6.A26, J7.A26, J8.A26
- net TONE 4: now also J2.A27, J3.A27, J4.A27, J5.A27, J6.A27, J7.A27, J8.A27; no longer J1.A28, J2.A28, J3.A28, J4.A28, J5.A28, J6.A28, J7.A28, J8.A28
- net TONE 5: now also J2.A29, J3.A29, J4.A29, J5.A29, J6.A29, J7.A29, J8.A29; no longer J1.A30, J2.A30, J3.A30, J4.A30, J5.A30, J6.A30, J7.A30, J8.A30
- net TONE 6: now also J2.A31, J3.A31, J4.A31, J5.A31, J6.A31, J7.A31, J8.A31; no longer J1.A32, J2.A32, J3.A32, J4.A32, J5.A32, J6.A32, J7.A32, J8.A32
- net TONE 7: now also J2.B21, J3.B21, J4.B21, J5.B21, J6.B21, J7.B21, J8.B21; no longer J2.B22, J3.B22, J4.B22, J5.B22, J6.B22, J7.B22, J8.B22
- net TONE 8: now also J2.B23, J3.B23, J4.B23, J5.B23, J6.B23, J7.B23, J8.B23; no longer J2.B24, J3.B24, J4.B24, J5.B24, J6.B24, J7.B24, J8.B24
- net TONE 9: now also J2.B25, J3.B25, J4.B25, J5.B25, J6.B25, J7.B25, J8.B25; no longer J2.B26, J3.B26, J4.B26, J5.B26, J6.B26, J7.B26, J8.B26
- new net SELECT 7: J2.A11, J3.A11, J4.A11, J5.A11, J6.A11, J7.A11, J8.A11
- new net SELECT 8: J2.A13, J3.A13, J4.A13, J5.A13, J6.A13, J7.A13, J8.A13
