File: Lyrebird Keyboard/Lyrebird Keyboard Piano Card/ENV 1-16.kicad_sch (KiCad schematic)
At the start: 224 parts

Commit message: Design Changes
Fix a number of symbol issues, and connection faults
Parts:
- C1, C11, C13, C15, C17, C18, C19, C20, C21, C22, C23, C24, C3, C5, C7, C9: footprint T491A -> SamacSys_Parts:T491A
- C10, C12, C14, C16, C2, C25, C26, C27, C28, C29, C30, C31, C32, C4, C6, C8: footprint CAPPM3528X210N -> SamacSys_Parts:CAPPM3528X210N
Changed lines of the file:
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@@
       (effects (font (size 1.27 1.27)) (justify left))
     )
-    (property "Footprint" "CAPPM3528X210N" (at 108.28 87.63 0)
+    (property "Footprint" "SamacSys_Parts:CAPPM3528X210N" (at 108.28 87.63 0)
       (effects (font (size 1.27 1.27)) (justify left top) hide)
     )
@@
       (effects (font (size 1.27 1.27)))
     )
-    (property "Footprint" "T491A" (at 184.15 423.85 0)
+    (property "Footprint" "SamacSys_Parts:T491A" (at 184.15 423.85 0)
       (effects (font (size 1.27 1.27)) (justify left top) hide)
     )
@@
       (effects (font (size 1.27 1.27)))
     )
-    (property "Footprint" "T491A" (at 46.99 381.94 0)
+    (property "Footprint" "SamacSys_Parts:T491A" (at 46.99 381.94 0)
       (effects (font (size 1.27 1.27)) (justify left top) hide)
     )
@@
       (effects (font (size 1.27 1.27)) (justify left))
     )
-    (property "Footprint" "CAPPM3528X210N" (at -30.15 264.16 0)
+    (property "Footprint" "SamacSys_Parts:CAPPM3528X210N" (at -30.15 264.16 0)
       (effects (font (size 1.27 1.27)) (justify left top) hide)
     )
@@
       (effects (font (size 1.27 1.27)))
     )
-    (property "Footprint" "T491A" (at 48.26 162.23 0)
+    (property "Footprint" "SamacSys_Parts:T491A" (at 48.26 162.23 0)
       (effects (font (size 1.27 1.27)) (justify left top) hide)
     )
@@
       (effects (font (size 1.27 1.27)) (justify left))
     )
-    (property "Footprint" "CAPPM3528X210N" (at 107.01 307.34 0)
+    (property "Footprint" "SamacSys_Parts:CAPPM3528X210N" (at 107.01 307.34 0)
       (effects (font (size 1.27 1.27)) (justify left top) hide)
     )
@@
       (effects (font (size 1.27 1.27)) (justify left))
     )
-    (property "Footprint" "CAPPM3528X210N" (at -30.15 307.34 0)
+    (property "Footprint" "SamacSys_Parts:CAPPM3528X210N" (at -30.15 307.34 0)
       (effects (font (size 1.27 1.27)) (justify left top) hide)
     )
@@
       (effects (font (size 1.27 1.27)))
     )
-    (property "Footprint" "T491A" (at 184.15 338.76 0)
+    (property "Footprint" "SamacSys_Parts:T491A" (at 184.15 338.76 0)
       (effects (font (size 1.27 1.27)) (justify left top) hide)
     )
@@
       (effects (font (size 1.27 1.27)))
     )
-    (property "Footprint" "T491A" (at 184.15 294.31 0)
+    (property "Footprint" "SamacSys_Parts:T491A" (at 184.15 294.31 0)
       (effects (font (size 1.27 1.27)) (justify left top) hide)
     )
@@
       (effects (font (size 1.27 1.27)) (justify left))
     )
-    (property "Footprint" "CAPPM3528X210N" (at 107.01 349.25 0)
+    (property "Footprint" "SamacSys_Parts:CAPPM3528X210N" (at 107.01 349.25 0)
       (effects (font (size 1.27 1.27)) (justify left top) hide)
     )
@@
       (effects (font (size 1.27 1.27)))
     )
-    (property "Footprint" "T491A" (at 185.42 119.05 0)
+    (property "Footprint" "SamacSys_Parts:T491A" (at 185.42 119.05 0)
       (effects (font (size 1.27 1.27)) (justify left top) hide)
     )
@@
       (effects (font (size 1.27 1.27)))
     )
-    (property "Footprint" "T491A" (at 46.99 249.86 0)
+    (property "Footprint" "SamacSys_Parts:T491A" (at 46.99 249.86 0)
       (effects (font (size 1.27 1.27)) (justify left top) hide)
     )
@@
       (effects (font (size 1.27 1.27)) (justify left))
     )
-    (property "Footprint" "CAPPM3528X210N" (at 107.01 264.16 0)
+    (property "Footprint" "SamacSys_Parts:CAPPM3528X210N" (at 107.01 264.16 0)
       (effects (font (size 1.27 1.27)) (justify left top) hide)
     )
@@
       (effects (font (size 1.27 1.27)))
     )
-    (property "Footprint" "T491A" (at 46.99 338.76 0)
+    (property "Footprint" "SamacSys_Parts:T491A" (at 46.99 338.76 0)
       (effects (font (size 1.27 1.27)) (justify left top) hide)
     )
@@
       (effects (font (size 1.27 1.27)))
     )
-    (property "Footprint" "T491A" (at 185.42 205.41 0)
+    (property "Footprint" "SamacSys_Parts:T491A" (at 185.42 205.41 0)
       (effects (font (size 1.27 1.27)) (justify left top) hide)
     )
@@
       (effects (font (size 1.27 1.27)) (justify left))
     )
-    (property "Footprint" "CAPPM3528X210N" (at -28.88 87.63 0)
+    (property "Footprint" "SamacSys_Parts:CAPPM3528X210N" (at -28.88 87.63 0)
       (effects (font (size 1.27 1.27)) (justify left top) hide)
     )
@@
       (effects (font (size 1.27 1.27)))
     )
-    (property "Footprint" "T491A" (at 184.15 249.86 0)
+    (property "Footprint" "SamacSys_Parts:T491A" (at 184.15 249.86 0)
       (effects (font (size 1.27 1.27)) (justify left top) hide)
     )
@@
       (effects (font (size 1.27 1.27)) (justify left))
     )
-    (property "Footprint" "CAPPM3528X210N" (at 107.01 219.71 0)
+    (property "Footprint" "SamacSys_Parts:CAPPM3528X210N" (at 107.01 219.71 0)
       (effects (font (size 1.27 1.27)) (justify left top) hide)
     )
@@
       (effects (font (size 1.27 1.27)))
     )
-    (property "Footprint" "T491A" (at 48.26 205.41 0)
+    (property "Footprint" "SamacSys_Parts:T491A" (at 48.26 205.41 0)
       (effects (font (size 1.27 1.27)) (justify left top) hide)
     )
@@
       (effects (font (size 1.27 1.27)) (justify left))
     )
-    (property "Footprint" "CAPPM3528X210N" (at 107.01 175.26 0)
+    (property "Footprint" "SamacSys_Parts:CAPPM3528X210N" (at 107.01 175.26 0)
       (effects (font (size 1.27 1.27)) (justify left top) hide)
     )
@@
       (effects (font (size 1.27 1.27)) (justify left))
     )
-    (property "Footprint" "CAPPM3528X210N" (at -30.15 219.71 0)
+    (property "Footprint" "SamacSys_Parts:CAPPM3528X210N" (at -30.15 219.71 0)
       (effects (font (size 1.27 1.27)) (justify left top) hide)
     )
@@
       (effects (font (size 1.27 1.27)) (justify left))
     )
-    (property "Footprint" "CAPPM3528X210N" (at -30.15 349.25 0)
+    (property "Footprint" "SamacSys_Parts:CAPPM3528X210N" (at -30.15 349.25 0)
       (effects (font (size 1.27 1.27)) (justify left top) hide)
     )
@@
       (effects (font (size 1.27 1.27)) (justify left))
     )
-    (property "Footprint" "CAPPM3528X210N" (at -30.15 175.26 0)
+    (property "Footprint" "SamacSys_Parts:CAPPM3528X210N" (at -30.15 175.26 0)
       (effects (font (size 1.27 1.27)) (justify left top) hide)
     )
@@
       (effects (font (size 1.27 1.27)))
     )
-    (property "Footprint" "T491A" (at 46.99 294.31 0)
+    (property "Footprint" "SamacSys_Parts:T491A" (at 46.99 294.31 0)
       (effects (font (size 1.27 1.27)) (justify left top) hide)
     )
@@
       (effects (font (size 1.27 1.27)))
     )
-    (property "Footprint" "T491A" (at 46.99 423.85 0)
+    (property "Footprint" "SamacSys_Parts:T491A" (at 46.99 423.85 0)
       (effects (font (size 1.27 1.27)) (justify left top) hide)
     )
@@
       (effects (font (size 1.27 1.27)))
     )
-    (property "Footprint" "T491A" (at 48.26 119.05 0)
+    (property "Footprint" "SamacSys_Parts:T491A" (at 48.26 119.05 0)
       (effects (font (size 1.27 1.27)) (justify left top) hide)
     )
@@
       (effects (font (size 1.27 1.27)))
     )
-    (property "Footprint" "T491A" (at 185.42 162.23 0)
+    (property "Footprint" "SamacSys_Parts:T491A" (at 185.42 162.23 0)
       (effects (font (size 1.27 1.27)) (justify left top) hide)
     )
@@
       (effects (font (size 1.27 1.27)) (justify left))
     )
-    (property "Footprint" "CAPPM3528X210N" (at -28.88 130.81 0)
+    (property "Footprint" "SamacSys_Parts:CAPPM3528X210N" (at -28.88 130.81 0)
       (effects (font (size 1.27 1.27)) (justify left top) hide)
     )
@@
       (effects (font (size 1.27 1.27)))
     )
-    (property "Footprint" "T491A" (at 184.15 381.94 0)
+    (property "Footprint" "SamacSys_Parts:T491A" (at 184.15 381.94 0)
       (effects (font (size 1.27 1.27)) (justify left top) hide)
     )
@@
       (effects (font (size 1.27 1.27)) (justify left))
     )
-    (property "Footprint" "CAPPM3528X210N" (at -28.88 44.45 0)
+    (property "Footprint" "SamacSys_Parts:CAPPM3528X210N" (at -28.88 44.45 0)
       (effects (font (size 1.27 1.27)) (justify left top) hide)
     )
@@
       (effects (font (size 1.27 1.27)) (justify left))
     )
-    (property "Footprint" "CAPPM3528X210N" (at 108.28 130.81 0)
+    (property "Footprint" "SamacSys_Parts:CAPPM3528X210N" (at 108.28 130.81 0)
       (effects (font (size 1.27 1.27)) (justify left top) hide)
     )
@@
       (effects (font (size 1.27 1.27)) (justify left))
     )
-    (property "Footprint" "CAPPM3528X210N" (at 108.28 44.45 0)
+    (property "Footprint" "SamacSys_Parts:CAPPM3528X210N" (at 108.28 44.45 0)
       (effects (font (size 1.27 1.27)) (justify left top) hide)
     )
