File: Lyrebird Keyboard/Lyrebird Keyboard Piano Card/ENV 17-34.kicad_sch (KiCad schematic)
At the start: 252 parts

Commit message: Design Changes
Fix a number of symbol issues, and connection faults
Parts:
- C17, C18, C19, C20, C21, C22, C23, C24: footprint T491A -> SamacSys_Parts:T491A
- C25, C26, C27, C28, C29, C30, C31, C32: footprint CAPPM3528X210N -> SamacSys_Parts:CAPPM3528X210N
Changed lines of the file:
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@@
       (effects (font (size 1.27 1.27)) (justify left))
     )
-    (property "Footprint" "CAPPM3528X210N" (at -32.69 378.46 0)
+    (property "Footprint" "SamacSys_Parts:CAPPM3528X210N" (at -32.69 378.46 0)
       (effects (font (size 1.27 1.27)) (justify left top) hide)
     )
@@
       (effects (font (size 1.27 1.27)))
     )
-    (property "Footprint" "T491A" (at 44.45 247.32 0)
+    (property "Footprint" "SamacSys_Parts:T491A" (at 44.45 247.32 0)
       (effects (font (size 1.27 1.27)) (justify left top) hide)
     )
@@
       (effects (font (size 1.27 1.27)))
     )
-    (property "Footprint" "T491A" (at 44.45 213.03 0)
+    (property "Footprint" "SamacSys_Parts:T491A" (at 44.45 213.03 0)
       (effects (font (size 1.27 1.27)) (justify left top) hide)
     )
@@
       (effects (font (size 1.27 1.27)) (justify left))
     )
-    (property "Footprint" "CAPPM3528X210N" (at -32.69 344.17 0)
+    (property "Footprint" "SamacSys_Parts:CAPPM3528X210N" (at -32.69 344.17 0)
       (effects (font (size 1.27 1.27)) (justify left top) hide)
     )
@@
       (effects (font (size 1.27 1.27)))
     )
-    (property "Footprint" "T491A" (at 44.45 281.61 0)
+    (property "Footprint" "SamacSys_Parts:T491A" (at 44.45 281.61 0)
       (effects (font (size 1.27 1.27)) (justify left top) hide)
     )
@@
       (effects (font (size 1.27 1.27)) (justify left))
     )
-    (property "Footprint" "CAPPM3528X210N" (at 109.55 172.72 0)
+    (property "Footprint" "SamacSys_Parts:CAPPM3528X210N" (at 109.55 172.72 0)
       (effects (font (size 1.27 1.27)) (justify left top) hide)
     )
@@
       (effects (font (size 1.27 1.27)) (justify left))
     )
-    (property "Footprint" "CAPPM3528X210N" (at -32.69 104.14 0)
+    (property "Footprint" "SamacSys_Parts:CAPPM3528X210N" (at -32.69 104.14 0)
       (effects (font (size 1.27 1.27)) (justify left top) hide)
     )
@@
       (effects (font (size 1.27 1.27)))
     )
-    (property "Footprint" "T491A" (at 186.69 385.75 0)
+    (property "Footprint" "SamacSys_Parts:T491A" (at 186.69 385.75 0)
       (effects (font (size 1.27 1.27)) (justify left top) hide)
     )
@@
       (effects (font (size 1.27 1.27)) (justify left))
     )
-    (property "Footprint" "CAPPM3528X210N" (at -32.69 172.72 0)
+    (property "Footprint" "SamacSys_Parts:CAPPM3528X210N" (at -32.69 172.72 0)
       (effects (font (size 1.27 1.27)) (justify left top) hide)
     )
@@
       (effects (font (size 1.27 1.27)))
     )
-    (property "Footprint" "T491A" (at 186.69 144.45 0)
+    (property "Footprint" "SamacSys_Parts:T491A" (at 186.69 144.45 0)
       (effects (font (size 1.27 1.27)) (justify left top) hide)
     )
@@
       (effects (font (size 1.27 1.27)) (justify left))
     )
-    (property "Footprint" "CAPPM3528X210N" (at -32.69 207.01 0)
+    (property "Footprint" "SamacSys_Parts:CAPPM3528X210N" (at -32.69 207.01 0)
       (effects (font (size 1.27 1.27)) (justify left top) hide)
     )
@@
       (effects (font (size 1.27 1.27)) (justify left))
     )
-    (property "Footprint" "CAPPM3528X210N" (at 109.55 104.14 0)
+    (property "Footprint" "SamacSys_Parts:CAPPM3528X210N" (at 109.55 104.14 0)
       (effects (font (size 1.27 1.27)) (justify left top) hide)
     )
@@
       (effects (font (size 1.27 1.27)))
     )
-    (property "Footprint" "T491A" (at 186.69 213.03 0)
+    (property "Footprint" "SamacSys_Parts:T491A" (at 186.69 213.03 0)
       (effects (font (size 1.27 1.27)) (justify left top) hide)
     )
@@
       (effects (font (size 1.27 1.27)) (justify left))
     )
-    (property "Footprint" "CAPPM3528X210N" (at 109.55 207.01 0)
+    (property "Footprint" "SamacSys_Parts:CAPPM3528X210N" (at 109.55 207.01 0)
       (effects (font (size 1.27 1.27)) (justify left top) hide)
     )
@@
       (effects (font (size 1.27 1.27)))
     )
-    (property "Footprint" "T491A" (at 44.45 350.19 0)
+    (property "Footprint" "SamacSys_Parts:T491A" (at 44.45 350.19 0)
       (effects (font (size 1.27 1.27)) (justify left top) hide)
     )
@@
       (effects (font (size 1.27 1.27)))
     )
-    (property "Footprint" "T491A" (at 44.45 453.06 0)
+    (property "Footprint" "SamacSys_Parts:T491A" (at 44.45 453.06 0)
       (effects (font (size 1.27 1.27)) (justify left top) hide)
     )
@@
       (effects (font (size 1.27 1.27)) (justify left))
     )
-    (property "Footprint" "CAPPM3528X210N" (at -32.69 241.3 0)
+    (property "Footprint" "SamacSys_Parts:CAPPM3528X210N" (at -32.69 241.3 0)
       (effects (font (size 1.27 1.27)) (justify left top) hide)
     )
@@
       (effects (font (size 1.27 1.27)) (justify left))
     )
-    (property "Footprint" "CAPPM3528X210N" (at 109.55 276.86 0)
+    (property "Footprint" "SamacSys_Parts:CAPPM3528X210N" (at 109.55 276.86 0)
       (effects (font (size 1.27 1.27)) (justify left top) hide)
     )
@@
       (effects (font (size 1.27 1.27)))
     )
-    (property "Footprint" "T491A" (at 44.45 144.45 0)
+    (property "Footprint" "SamacSys_Parts:T491A" (at 44.45 144.45 0)
       (effects (font (size 1.27 1.27)) (justify left top) hide)
     )
@@
       (effects (font (size 1.27 1.27)))
     )
-    (property "Footprint" "T491A" (at 44.45 315.9 0)
+    (property "Footprint" "SamacSys_Parts:T491A" (at 44.45 315.9 0)
       (effects (font (size 1.27 1.27)) (justify left top) hide)
     )
@@
       (effects (font (size 1.27 1.27)) (justify left))
     )
-    (property "Footprint" "CAPPM3528X210N" (at 109.55 69.85 0)
+    (property "Footprint" "SamacSys_Parts:CAPPM3528X210N" (at 109.55 69.85 0)
       (effects (font (size 1.27 1.27)) (justify left top) hide)
     )
@@
       (effects (font (size 1.27 1.27)) (justify left))
     )
-    (property "Footprint" "CAPPM3528X210N" (at 109.55 241.3 0)
+    (property "Footprint" "SamacSys_Parts:CAPPM3528X210N" (at 109.55 241.3 0)
       (effects (font (size 1.27 1.27)) (justify left top) hide)
     )
@@
       (effects (font (size 1.27 1.27)))
     )
-    (property "Footprint" "T491A" (at 44.45 418.77 0)
+    (property "Footprint" "SamacSys_Parts:T491A" (at 44.45 418.77 0)
       (effects (font (size 1.27 1.27)) (justify left top) hide)
     )
@@
       (effects (font (size 1.27 1.27)))
     )
-    (property "Footprint" "T491A" (at 44.45 384.48 0)
+    (property "Footprint" "SamacSys_Parts:T491A" (at 44.45 384.48 0)
       (effects (font (size 1.27 1.27)) (justify left top) hide)
     )
@@
       (effects (font (size 1.27 1.27)) (justify left))
     )
-    (property "Footprint" "CAPPM3528X210N" (at -32.69 138.43 0)
+    (property "Footprint" "SamacSys_Parts:CAPPM3528X210N" (at -32.69 138.43 0)
       (effects (font (size 1.27 1.27)) (justify left top) hide)
     )
@@
       (effects (font (size 1.27 1.27)))
     )
-    (property "Footprint" "T491A" (at 44.45 178.74 0)
+    (property "Footprint" "SamacSys_Parts:T491A" (at 44.45 178.74 0)
       (effects (font (size 1.27 1.27)) (justify left top) hide)
     )
@@
       (effects (font (size 1.27 1.27)) (justify left))
     )
-    (property "Footprint" "CAPPM3528X210N" (at 109.55 311.15 0)
+    (property "Footprint" "SamacSys_Parts:CAPPM3528X210N" (at 109.55 311.15 0)
       (effects (font (size 1.27 1.27)) (justify left top) hide)
     )
@@
       (effects (font (size 1.27 1.27)))
     )
-    (property "Footprint" "T491A" (at 186.69 351.46 0)
+    (property "Footprint" "SamacSys_Parts:T491A" (at 186.69 351.46 0)
       (effects (font (size 1.27 1.27)) (justify left top) hide)
     )
@@
       (effects (font (size 1.27 1.27)) (justify left))
     )
-    (property "Footprint" "CAPPM3528X210N" (at -32.69 69.85 0)
+    (property "Footprint" "SamacSys_Parts:CAPPM3528X210N" (at -32.69 69.85 0)
       (effects (font (size 1.27 1.27)) (justify left top) hide)
     )
@@
       (effects (font (size 1.27 1.27)) (justify left))
     )
-    (property "Footprint" "CAPPM3528X210N" (at 109.55 138.43 0)
+    (property "Footprint" "SamacSys_Parts:CAPPM3528X210N" (at 109.55 138.43 0)
       (effects (font (size 1.27 1.27)) (justify left top) hide)
     )
@@
       (effects (font (size 1.27 1.27)))
     )
-    (property "Footprint" "T491A" (at 186.69 281.61 0)
+    (property "Footprint" "SamacSys_Parts:T491A" (at 186.69 281.61 0)
       (effects (font (size 1.27 1.27)) (justify left top) hide)
     )
@@
       (effects (font (size 1.27 1.27)))
     )
-    (property "Footprint" "T491A" (at 186.69 247.32 0)
+    (property "Footprint" "SamacSys_Parts:T491A" (at 186.69 247.32 0)
       (effects (font (size 1.27 1.27)) (justify left top) hide)
     )
@@
       (effects (font (size 1.27 1.27)) (justify left))
     )
-    (property "Footprint" "CAPPM3528X210N" (at -32.69 275.59 0)
+    (property "Footprint" "SamacSys_Parts:CAPPM3528X210N" (at -32.69 275.59 0)
       (effects (font (size 1.27 1.27)) (justify left top) hide)
     )
@@
       (effects (font (size 1.27 1.27)))
     )
-    (property "Footprint" "T491A" (at 186.69 315.9 0)
+    (property "Footprint" "SamacSys_Parts:T491A" (at 186.69 315.9 0)
       (effects (font (size 1.27 1.27)) (justify left top) hide)
     )
@@
       (effects (font (size 1.27 1.27)))
     )
-    (property "Footprint" "T491A" (at 186.69 178.74 0)
+    (property "Footprint" "SamacSys_Parts:T491A" (at 186.69 178.74 0)
       (effects (font (size 1.27 1.27)) (justify left top) hide)
     )
@@
       (effects (font (size 1.27 1.27)) (justify left))
     )
-    (property "Footprint" "CAPPM3528X210N" (at -32.69 309.88 0)
+    (property "Footprint" "SamacSys_Parts:CAPPM3528X210N" (at -32.69 309.88 0)
       (effects (font (size 1.27 1.27)) (justify left top) hide)
     )
