File: Lyrebird Keyboard/Lyrebird Keyboard Piano Card/ENV 35-52.kicad_sch (KiCad schematic)
At the start: 252 parts

Commit message: Design Changes
Fix a number of symbol issues, and connection faults
Parts:
- C17, C18, C19, C20, C21, C22, C23, C24: footprint T491A -> SamacSys_Parts:T491A
- C25, C26, C27, C28, C29, C30, C31, C32: footprint CAPPM3528X210N -> SamacSys_Parts:CAPPM3528X210N
- R82: value 220k -> 180k
- R82: value 180k -> 120k
Connections:
- net G#40S: now reaches R82.1, R82.2
- net F37S: now reaches R82.1, R82.2
- net F49: now reaches C20.1 (+), R82.2, R82.2
- net F#38: now reaches C17.1 (+), R82.2, R82.2
- net A#42: now reaches C21.1 (+), R82.2, R82.2
- net D#47: now reaches C18.1 (+), R82.2, R82.2
- net G39: now reaches C18.1 (+), R82.2, R82.2
- net F49S: now reaches R82.1, R82.2
- net G#52: now reaches C21.1 (+), R82.2, R82.2
- net F#50: now reaches C21.1 (+), R82.2, R82.2
- net C#45: now reaches C24.1 (+), R82.2, R82.2
- net D46: now reaches C17.1 (+), R82.2, R82.2
- net A41: now reaches C20.1 (+), R82.2, R82.2
- net G#40: now reaches C19.1 (+), R82.2, R82.2
- net B43S: now reaches R82.1, R82.2
- net D#35S: now reaches R82.1, R82.2
- net C44S: now reaches R82.1, R82.2
- net A41S: now reaches R82.1, R82.2
- net E48S: now reaches R82.1, R82.2
- net C44: now reaches C23.1 (+), R82.2, R82.2
- net G51: now reaches C21.1 (+), R82.2, R82.2
- net F#50S: now reaches R82.1, R82.2
- net D#47S: now reaches R82.1, R82.2
- net C#45S: now reaches R82.1, R82.2
- net B43: now reaches C22.1 (+), R82.2, R82.2
- net G51S: now reaches R82.1, R82.2
- net F#38S: now reaches R82.1, R82.2
- net G#52S: now reaches R82.1, R82.2
- net G39S: now reaches R82.1, R82.2
- net E48: now reaches C19.1 (+), R82.2, R82.2
- net E36S: now reaches R82.1, R82.2
- net A#42S: now reaches R82.1, R82.2
- net D46S: now reaches R82.1, R82.2
