File: Lyrebird Keyboard/Lyrebird Keyboard Piano Card/Lyrebird Keyboard Piano Card.kicad_sch (KiCad schematic)
At the start: 1 part, among them J1 Edge Connector

Commit message: Design Changes
Fix a number of symbol issues, and connection faults
Parts:
- added C147, C148, C149, C150, C151, C152: C1206C104J3RACTU, SamacSys_Parts:C1206, symbol SamacSys_Parts:C1206C104J3RACTU
- added C153, C154: 16TZV100M6.3X6.1, SamacSys_Parts:16TZV100M63X61, symbol SamacSys_Parts:16TZV100M6.3X6.1
- added C44 (x4): 100nF, Capacitor_SMD:C_1206_3216Metric, symbol Device:C_Small
- added C44 (x2): 47nF, Capacitor_SMD:C_1206_3216Metric, symbol Device:C_Small
- added C44 (x10): 10nF, Capacitor_SMD:C_1206_3216Metric, symbol Device:C_Small
- added C44 (x9): 22nF, Capacitor_SMD:C_1206_3216Metric, symbol Device:C_Small
- added C44 (x9): 1nF, Capacitor_SMD:C_1206_3216Metric, symbol Device:C_Small
- added C44 (x2): 220nF, Capacitor_SMD:C_1206_3216Metric, symbol Device:C_Small
- added C44 (x3): 2.2nF, Capacitor_SMD:C_1206_3216Metric, symbol Device:C_Small
- added C44 (x4): 4.7nF, Capacitor_SMD:C_1206_3216Metric, symbol Device:C_Small
- added C44: 100pF, Capacitor_SMD:C_1206_3216Metric, symbol Device:C_Small
- added C44: 150nF, Capacitor_SMD:C_1206_3216Metric, symbol Device:C_Small
- added C44: 1.5nF, Capacitor_SMD:C_1206_3216Metric, symbol Device:C_Small
- added C44: 68pF, Capacitor_SMD:C_1206_3216Metric, symbol Device:C_Small
- added C44 (x2): 15nF, Capacitor_SMD:C_1206_3216Metric, symbol Device:C_Small
- added C44: 470pF, Capacitor_SMD:C_1206_3216Metric, symbol Device:C_Small
- added C44: 680pF, Capacitor_SMD:C_1206_3216Metric, symbol Device:C_Small
- added C44 (x2): 6.8nF, Capacitor_SMD:C_1206_3216Metric, symbol Device:C_Small
- added D207 (x5): 1N4148W, Diode_SMD:D_SOD-123, symbol Diode:1N4148W
- added IC4: NE5517DR2G, NE5517:SOIC-16_ONS, symbol NE5517:NE5517DR2G
- added IC5, IC8: LF347DT, SamacSys_Parts:SOIC127P600X175-14N, symbol SamacSys_Parts:LF347DT
- added IC6: SN74LVC00APWR, SamacSys_Parts:SOP65P640X120-14N, symbol SamacSys_Parts:SN74LVC00APWR
- added IC7, IC9: ~, symbol SamacSys_Parts:MN3009
- added J2: Harpsichord Select, symbol Connector:Conn_01x01_Pin
- added J3: Normal Select, symbol Connector:Conn_01x01_Pin
- added J4: Bright Select, symbol Connector:Conn_01x01_Pin
- added J5: Mellow Select, symbol Connector:Conn_01x01_Pin
- added R82 (x10): 27k, Resistor_SMD:R_1206_3216Metric, symbol Device:R
- added R82 (x2): 68k, Resistor_SMD:R_1206_3216Metric, symbol Device:R
- added R82 (x5): 15k, Resistor_SMD:R_1206_3216Metric, symbol Device:R
- added R82 (x6): 10k, Resistor_SMD:R_1206_3216Metric, symbol Device:R
- added R82 (x9): 33k, Resistor_SMD:R_1206_3216Metric, symbol Device:R
- added R82 (x7): 22k, Resistor_SMD:R_1206_3216Metric, symbol Device:R
- added R82 (x6): 270k, Resistor_SMD:R_1206_3216Metric, symbol Device:R
- added R82 (x2): 1k, Resistor_SMD:R_1206_3216Metric, symbol Device:R
- added R82 (x17): 47k, Resistor_SMD:R_1206_3216Metric, symbol Device:R
- added R82 (x5): 12k, Resistor_SMD:R_1206_3216Metric, symbol Device:R
- added R82: 150k, Resistor_SMD:R_1206_3216Metric, symbol Device:R
- added R82 (x5): 39k, Resistor_SMD:R_1206_3216Metric, symbol Device:R
- added R82 (x2): 220R, Resistor_SMD:R_1206_3216Metric, symbol Device:R
- added R82 (x2): 120k, Resistor_SMD:R_1206_3216Metric, symbol Device:R
- added R82: 56k, Resistor_SMD:R_1206_3216Metric, symbol Device:R
- added R82 (x2): 82k, Resistor_SMD:R_1206_3216Metric, symbol Device:R
- added U1, U2, U3: LF347DT, SamacSys_Parts:SOIC127P600X175-14N, symbol SamacSys_Parts:LF347DT-PF
- added VR1, VR2, VR3: 22k, 3214W1205E, symbol SamacSys_Parts:3214W-1-223E
- added VR4, VR5: 3214W-1-223E, SamacSys_Parts:3214W1205E, symbol SamacSys_Parts:3214W-1-223E
- added VR6: 3313J-1-473E, SamacSys_Parts:3313J-1, symbol SamacSys_Parts:3313J-1-473E
Connections:
- net +15V: now also C147.2, IC5.4 (VCC+), IC8.4 (VCC+), R82.2
- net -15V: now also C148.1, IC5.11 (VCC-), IC6.7 (GND), IC7.5 (Vdd), IC8.11 (VCC-), IC9.5 (Vdd), R82.1, R82.1, R82.2
- net GND: now also C147.1, C148.2, C149.2, C150.1, C151.2, C152.1, C153.2 (-), C154.1 (+), C44.1, C44.1, C44.1, C44.1, C44.1, C44.1, C44.1, C44.1, C44.1, C44.1, C44.1, C44.1, C44.2, IC7.1 (GND), IC9.1 (GND), R82.1, R82.1, R82.1, R82.1, R82.1, R82.2, R82.2, U1.10 (+), U1.12 (+), U1.3 (+), VR1.2, VR1.3, VR2.2, VR2.3, VR3.2, VR3.3, VR4.2 (WIPER), VR4.3 (CW), VR5.2 (WIPER), VR5.3 (CW), VR6.1, VR6.2
- new net: C44.2, R82.2 (x13)
- new net: C44.2, R82.1, R82.2 (x13)
- new net: C44.1, R82.1, R82.2
- new net: C44.2, R82.2, R82.2, R82.2
- new net: C44.1, C44.1, D207.1 (K), R82.2 (x5)
- new net: C44.1, C44.2, VR3.1
- new net: C44.1, C44.2, VR6.3
- new net: IC7.8 (OUT1), IC9.3 (IN)
- new net: IC9.4 (Vgg), R82.1, R82.2
- new net: C44.1, R82.1, R82.1, R82.1, R82.1, R82.1
- new net: C44.2, R82.1, R82.2, R82.2, R82.2 (x5)
- new net: J4.1 (Pin_1), R82.1, R82.2
- new net: C44.1, C44.1, R82.1, R82.1, U1.14
- new net: C44.1, C44.2, VR2.1
- new net: C44.2, R82.1, R82.2, R82.2, U1.9 (-)
- new net: C44.1, R82.1, R82.1, R82.1, R82.1, R82.1, R82.1 (x2)
- new net: C44.2, R82.1, R82.2, R82.2, U1.2 (-)
- new net: C44.1, C44.2, VR5.1 (CCW)
- new net: C44.2, R82.1, R82.2, R82.2, U1.13 (-)
- new net: C44.1, C44.1, R82.1, R82.1, U1.8
- new net: IC7.4 (Vgg), R82.1, R82.2
- new net: R82.1, R82.1, R82.1
- new net: J3.1 (Pin_1), R82.1, R82.2
- new net: C44.1, C44.1, R82.1, R82.1, U1.1
- new net: C44.1, R82.1
- new net: J5.1 (Pin_1), R82.1, R82.2
- new net: J2.1 (Pin_1), R82.1, R82.2
- new net: C44.1, C44.2, VR4.1 (CCW)
- new net: C44.1, C44.2, VR1.1
- new net +15V IC1,2,3,4: C150.2, C152.2, C153.1 (+), IC4.11 (V+), R82.1
- new net -15V IC1,2,3,4: C149.1, C151.1, C154.2 (-), IC4.6 (V-), R82.1
- new net BBD IN: IC7.3 (IN)
- new net BBD OUT: IC9.7 (OUT2), IC9.8 (OUT1)
- new net INPUT 4: C44.2, R82.1, R82.2, R82.2
- new net INPUT 5: C44.2, R82.1, R82.2, R82.2
- new net INPUT BRIGHT: C44.1, C44.2, R82.2
- new net INPUT CMB: C44.2, R82.1, R82.1, R82.2, R82.2
- new net INPUT H.CHORD: C44.1, C44.2, R82.2
- new net INPUT MELLOW: C44.1, C44.2, R82.2
- new net INPUT NORMAL: C44.1, C44.2, R82.2
- new net MIX OUT: R82.1, R82.1, R82.1, R82.1
- new net NAND CLK 1: IC7.2 (CP1), IC9.2 (CP1)
- new net NAND CLK 2: IC7.6 (CP2), IC9.6 (CP2)
- new net OPAMP OUT1a: C44.1
- new net OPAMP OUT1b: C44.1, C44.1, C44.1, R82.1, R82.1
- new net OPAMP OUT1c: R82.2
- new net OPAMP OUT1d: R82.2
- new net OPAMP OUT2a: C44.1, C44.1, C44.1, R82.1, R82.1
- new net OPAMP OUT2b: C44.1, C44.1, C44.1, R82.1, R82.1
- new net OPAMP OUT2c: C44.2, R82.1, R82.2
- new net OPAMP OUT2d: C44.2, R82.1, R82.2
- new net OPAMP OUT3c: C44.2, R82.1, R82.2
- new net OPAMP OUT3d: C44.2, R82.1, R82.2
- new net OUTPUT 1: D207.2 (A)
- new net OUTPUT 2: D207.2 (A)
- new net OUTPUT 3: D207.2 (A)
- new net OUTPUT 4: D207.2 (A)
- new net OUTPUT 5: D207.2 (A)
- no-connect marks 0 -> 11
Other:
- added sheet Notes 53 to 70 (ENV 53-70.kicad_sch)
- added sheet Notes 71 to 73 (ENV 71-73.kicad_sch)

Commit message: Schematic Updates
Made updates to schematics, to use correct symbols, and minor PCB updates, further work on the piano card design
Parts:
- removed IC4: NE5517DR2G, NE5517:SOIC-16_ONS, symbol NE5517:NE5517DR2G
- removed IC5, IC8: LF347DT, SamacSys_Parts:SOIC127P600X175-14N, symbol SamacSys_Parts:LF347DT
- removed IC6: SN74LVC00APWR, SamacSys_Parts:SOP65P640X120-14N, symbol SamacSys_Parts:SN74LVC00APWR
- removed IC7, IC9: ~, symbol SamacSys_Parts:MN3009
- removed R82 (x2): 1k, Resistor_SMD:R_1206_3216Metric, symbol Device:R
- removed R82 (x2): 15k, Resistor_SMD:R_1206_3216Metric, symbol Device:R
- removed unit 2 of U3
- removed unit 1 of U3
- removed VR6: 3313J-1-473E, SamacSys_Parts:3313J-1, symbol SamacSys_Parts:3313J-1-473E
- added U6: 4011, symbol 4xxx:4011
- added U8: LF347DT, SamacSys_Parts:SOIC127P600X175-14N, symbol SamacSys_Parts:LF347DT-PF
- added VR6: 47k, 3214W1205E, symbol SamacSys_Parts:3214W-1-223E
- VR4, VR5: value 3214W-1-223E -> 22k; footprint SamacSys_Parts:3214W1205E -> 3214W1205E
Connections:
- net INPUT 4 is gone; now on an unnamed net: C44.2, R82.1, R82.2, R82.2
- net INPUT 5 is gone; now on an unnamed net: C44.2, R82.1, R82.2, R82.2
- net INPUT BRIGHT is gone; now on an unnamed net: C44.1, C44.2, R82.2
- net INPUT CMB is gone; now on an unnamed net: C44.2, R82.1, R82.1, R82.2, R82.2
- net INPUT H.CHORD is gone; now on an unnamed net: C44.1, C44.2, R82.2
- net INPUT MELLOW is gone; now on an unnamed net: C44.1, C44.2, R82.2
- net INPUT NORMAL is gone; now on an unnamed net: C44.1, C44.2, R82.2
- net OPAMP OUT1a is gone; now on an unnamed net: C44.1
- net OPAMP OUT1b is gone; now on an unnamed net: C44.1, C44.1, C44.1, R82.1, R82.1
- net OPAMP OUT1c is gone; now on an unnamed net: R82.2
- net OPAMP OUT1d is gone; now on an unnamed net: R82.2
- net OPAMP OUT2a is gone; now on an unnamed net: C44.1, C44.1, C44.1, R82.1, R82.1
- net OPAMP OUT2b is gone; now on an unnamed net: C44.1, C44.1, C44.1, R82.1, R82.1
- net OPAMP OUT2c is gone; now on an unnamed net: C44.2, R82.1, R82.2
- net OPAMP OUT2d is gone; now on an unnamed net: C44.2, R82.1, R82.2
- net OPAMP OUT3c is gone; now on an unnamed net: C44.2, R82.1, R82.2
- net OPAMP OUT3d is gone; now on an unnamed net: C44.2, R82.1, R82.2
- net GND: now also U1.5 (+), U2.10 (+), U2.12 (+), U2.3 (+), U2.5 (+), U3.10 (+), U3.12 (+), VR6.2, VR6.3
- net at C44.1, C44.2: now also VR6.1
- net at R82.1, R82.1, R82.1: now also U2.6 (-)
- no-connect marks 11 -> 0
Other:
- added sheet Effects and Pedals (EFFECTS.kicad_sch)
- moved on the sheet: C44, D207, J2, J3, J4, J5, R82, U1B, U2A, U2B, U2C, U2D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
