File: Lyrebird Keyboard/Lyrebird Keyboard Interconnect Mainboard/Lyrebird Keyboard Interconnect Mainboard.kicad_pcb (KiCad board)
At the start: 4 copper layers, 220.1 x 160.3 mm, 15 parts, among them J1 INSTMNT 4 (MIDI), J13 Keys 1 to 14, J14 Keys 15 to 28, J15 Keys 29 to 36, J16 Keys 37 to 45, J17 Keys 46 to 59, J18 Keys 60 to 73, J2 INSTMNT 3, J25 Pedals, J3 INSTMNT 2, J4 INSTMNT 1, J5 TONE SRC 4, J6 TONE SRC 3, J7 TONE SRC 2, J8 TONE SRC 1

Commit message: Updates
Parts:
- added J10: -15V, SamacSys_Parts:17761192, F.Cu at (-24.2, 37.2)
- added J11: 30V, SamacSys_Parts:17761192, F.Cu at (-24.2, 48.5)
- added J12: +VT, SamacSys_Parts:17761192, F.Cu at (-24.2, 59.8)
- added J26: +VED, SamacSys_Parts:17761192, F.Cu at (-24.2, 71.1)
- added J9: +15V, SamacSys_Parts:17761192, F.Cu at (-24.2, 25.9)
- J13, J14, J15, J16, J17, J18: moved to F.Cu
- moved J15 158.5 mm to (67.9, 108.1), turned to 90 degrees
- moved J14 128.3 mm to (100.0, 108.1), turned to 90 degrees
- moved J25 110.1 mm to (7.42, 28.3)
- moved J13 108.1 mm to (132.0, 108.1), turned to 90 degrees
- moved J16 60.3 mm to (84.0, 108.1)
- moved J18 42.2 mm to (148.1, 108.1)
- moved J1 39.7 mm to (250.0, 26.2)
- moved J2 39.7 mm to (224.5, 26.2)
- moved J3 39.7 mm to (199.3, 26.2)
- moved J4 39.7 mm to (173.8, 26.2)
- moved J5 39.7 mm to (148.5, 26.3)
- moved J8 39.7 mm to (72.2, 26.2)
- moved J7 39.7 mm to (97.7, 26.2)
- moved J6 39.7 mm to (123.1, 26.2)
- moved J17 27.5 mm to (116.0, 108.1)
Routing:
- net +30V: track 11.4 -> 595.2 mm
- net +15V: track 0.00 -> 540.8 mm
- net -15V: track 0.00 -> 412.0 mm
- net EXP 5: track 0.00 -> 183.4 mm
- net EXP 13: track 0.00 -> 183.4 mm
- net SELECT 7: track 0.00 -> 183.4 mm
- net TONE 8: track 0.00 -> 183.4 mm
- net EXP9: track 0.00 -> 183.4 mm
- net +VED: track 0.00 -> 183.4 mm
- net SUSTAIN: track 0.00 -> 183.4 mm
- net TONE 7: track 0.00 -> 183.4 mm
- net TONE 4: track 0.00 -> 183.4 mm
- net EXP8: track 0.00 -> 183.4 mm
- net TONE 11: track 0.00 -> 183.4 mm
- net EXP10: track 0.00 -> 183.4 mm
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Other:
- board size 220.1 x 160.3 mm -> 207.3 x 100.9 mm
- board text removed: "Soft"
- board text removed: "Sub In Level"
- board text removed: "Sustain"
